File: PCB/Blare.kicad_sch (KiCad schematic)
At the start: 11 parts, among them J1 Conn_01x08_Pin, SW1 SW_Push, SW2 SW_Push, SW3 SW_Push, SW4 SW_Push, U1 XIAO-ESP32-C3-SMD

Commit message: Complete all except BOM
Changed lines of the file:
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@@
 	(paper "A4")
+	(junction
+		(at 129.54 85.09)
+		(diameter 0)
+		(color 0 0 0 0)
+	)
 	(junction
 		(at 43.18 85.09)
@@
 	(junction
 		(at 43.18 105.41)
+		(diameter 0)
+		(color 0 0 0 0)
+	)
+	(junction
+		(at 130.81 88.9)
 		(diameter 0)
 		(color 0 0 0 0)
@@
 			)
 			(justify left bottom)
+		)
+	)
+	(symbol
+		(lib_id "power:PWR_FLAG")
+		(at 129.54 85.09 0)
+		(unit 1)
+		(body_style 1)
+		(exclude_from_sim no)
+		(in_bom yes)
+		(on_board yes)
+		(in_pos_files yes)
+		(dnp no)
+		(property "Reference" "#FLG01"
+			(at 129.54 83.185 0)
+			(hide yes)
+			(show_name no)
+			(do_not_autoplace no)
+			(effects
+				(font
+					(size 1.27 1.27)
+				)
+			)
+		)
+		(property "Value" "PWR_FLAG"
+			(at 129.286 80.772 0)
+			(show_name no)
+			(do_not_autoplace no)
+			(effects
+				(font
+					(size 1.27 1.27)
+				)
+				(justify left)
+			)
+		)
+		(property "Footprint" "Package_SO:TSSOP-28_4.4x9.7mm_P0.65mm"
+			(at 129.54 85.09 0)
+			(hide yes)
+			(show_name no)
+			(do_not_autoplace no)
+			(effects
+				(font
+					(size 1.27 1.27)
+				)
+			)
+		)
+		(property "Datasheet" ""
+			(at 129.54 85.09 0)
+			(hide yes)
+			(show_name no)
+			(do_not_autoplace no)
+			(effects
+				(font
+					(size 1.27 1.27)
+				)
+			)
+		)
+		(property "Description" "Special symbol for telling ERC where power comes from"
+			(at 129.54 85.09 0)
+			(hide yes)
+			(show_name no)
+			(do_not_autoplace no)
+			(effects
+				(font
+					(size 1.27 1.27)
+				)
+			)
+		)
+		(pin "1"
+		)
+		(instances
+			(project "Blare"
+				(path "/7dcd853a-b2fe-4ea9-a053-0232d1e8e6bb"
+					(reference "#FLG01")
+					(unit 1)
+				)
+			)
 		)
 	)
@@
 		)
 		(instances
-			(project "blare"
+			(project "Blare"
 				(path "/7dcd853a-b2fe-4ea9-a053-0232d1e8e6bb"
 					(reference "#PWR04")
@@
 		)
 		(instances
-			(project "blare"
+			(project "Blare"
 				(path "/7dcd853a-b2fe-4ea9-a053-0232d1e8e6bb"
 					(reference "H4")
@@
 		(in_pos_files yes)
 		(dnp no)
-		(fields_autoplaced yes)
 		(property "Reference" "#PWR07"
 			(at 135.89 85.09 0)
@@
 		)
 		(property "Value" "GND"
-			(at 133.35 85.0899 90)
+			(at 136.398 85.344 90)
 			(show_name no)
 			(do_not_autoplace no)
@@
 		)
 		(instances
-			(project "blare"
+			(project "Blare"
 				(path "/7dcd853a-b2fe-4ea9-a053-0232d1e8e6bb"
 					(reference "#PWR07")
@@
 		)
 		(instances
-			(project "blare"
+			(project "Blare"
 				(path "/7dcd853a-b2fe-4ea9-a053-0232d1e8e6bb"
 					(reference "#PWR03")
@@
 		)
 		(instances
-			(project "blare"
+			(project "Blare"
 				(path "/7dcd853a-b2fe-4ea9-a053-0232d1e8e6bb"
 					(reference "SW4")
@@
 		)
 		(instances
-			(project "blare"
+			(project "Blare"
 				(path "/7dcd853a-b2fe-4ea9-a053-0232d1e8e6bb"
 					(reference "SW3")
@@
 		)
 		(instances
-			(project "blare"
+			(project "Blare"
 				(path "/7dcd853a-b2fe-4ea9-a053-0232d1e8e6bb"
 					(reference "#PWR02")
@@
 		)
 		(instances
-			(project "blare"
+			(project "Blare"
 				(path "/7dcd853a-b2fe-4ea9-a053-0232d1e8e6bb"
 					(reference "#PWR08")
@@
 		)
 		(instances
-			(project "blare"
+			(project "Blare"
 				(path "/7dcd853a-b2fe-4ea9-a053-0232d1e8e6bb"
 					(reference "SW2")
@@
 		)
 		(instances
-			(project "blare"
+			(project "Blare"
 				(path "/7dcd853a-b2fe-4ea9-a053-0232d1e8e6bb"
 					(reference "H1")
@@
 		)
 		(instances
-			(project "blare"
+			(project "Blare"
 				(path "/7dcd853a-b2fe-4ea9-a053-0232d1e8e6bb"
 					(reference "H2")
@@
 		)
 		(instances
-			(project "blare"
+			(project "Blare"
 				(path "/7dcd853a-b2fe-4ea9-a053-0232d1e8e6bb"
 					(reference "BZ1")
@@
 		)
 		(instances
-			(project "blare"
+			(project "Blare"
 				(path "/7dcd853a-b2fe-4ea9-a053-0232d1e8e6bb"
 					(reference "#PWR01")
@@
 		)
 		(instances
-			(project "blare"
+			(project "Blare"
 				(path "/7dcd853a-b2fe-4ea9-a053-0232d1e8e6bb"
 					(reference "U1")
@@
 		)
 		(instances
-			(project "blare"
+			(project "Blare"
 				(path "/7dcd853a-b2fe-4ea9-a053-0232d1e8e6bb"
 					(reference "H3")
@@
 		)
 		(instances
-			(project "blare"
+			(project "Blare"
 				(path "/7dcd853a-b2fe-4ea9-a053-0232d1e8e6bb"
 					(reference "#PWR06")
@@
 		)
 		(instances
-			(project "blare"
+			(project "Blare"
 				(path "/7dcd853a-b2fe-4ea9-a053-0232d1e8e6bb"
 					(reference "SW1")
+					(unit 1)
+				)
+			)
+		)
+	)
+	(symbol
+		(lib_id "power:PWR_FLAG")
+		(at 130.81 88.9 0)
+		(unit 1)
+		(body_style 1)
+		(exclude_from_sim no)
+		(in_bom yes)
+		(on_board yes)
+		(in_pos_files yes)
+		(dnp no)
+		(fields_autoplaced yes)
+		(property "Reference" "#FLG02"
+			(at 130.81 86.995 0)
+			(hide yes)
+			(show_name no)
+			(do_not_autoplace no)
+			(effects
+				(font
+					(size 1.27 1.27)
+				)
+			)
+		)
+		(property "Value" "PWR_FLAG"
+			(at 130.81 83.82 0)
+			(show_name no)
+			(do_not_autoplace no)
+			(effects
+				(font
+					(size 1.27 1.27)
+				)
+			)
+		)
+		(property "Footprint" "Package_SO:TSSOP-28_4.4x9.7mm_P0.65mm"
+			(at 130.81 88.9 0)
+			(hide yes)
+			(show_name no)
+			(do_not_autoplace no)
+			(effects
+				(font
+					(size 1.27 1.27)
+				)
+			)
+		)
+		(property "Datasheet" ""
+			(at 130.81 88.9 0)
+			(hide yes)
+			(show_name no)
+			(do_not_autoplace no)
+			(effects
+				(font
+					(size 1.27 1.27)
+				)
+			)
+		)
+		(property "Description" "Special symbol for telling ERC where power comes from"
+			(at 130.81 88.9 0)
+			(hide yes)
+			(show_name no)
+			(do_not_autoplace no)
+			(effects
+				(font
+					(size 1.27 1.27)
+				)
+			)
+		)
+		(pin "1"
+		)
+		(instances
+			(project "Blare"
+				(path "/7dcd853a-b2fe-4ea9-a053-0232d1e8e6bb"
+					(reference "#FLG02")
 					(unit 1)
 				)
@@
 		)
 		(instances
-			(project "blare"
+			(project "Blare"
 				(path "/7dcd853a-b2fe-4ea9-a053-0232d1e8e6bb"
 					(reference "J1")
@@
 		)
 		(instances
-			(project "blare"
+			(project "Blare"
 				(path "/7dcd853a-b2fe-4ea9-a053-0232d1e8e6bb"
 					(reference "#PWR05")
